File: cortrace-connector/cortrace-connector.kicad_sch (KiCad schematic)
At the start: 8 parts, among them J1 FPGA-PORT, J2 Conn_ARM_Cortex_Debug_ETM_20, J4 SWD-PORT

Commit message: feat(connector): use a 1.27 mm SMD female socket for the TRACE port
Swap J2 from the pin header footprint to the stock KiCad PinSocket_2x10_P1.27mm_Vertical_SMD. Its pads are already numbered mirrored, so the back-side placement needs no pad swap and the footprint matches the library again.
Parts:
- J2: footprint Connector_PinHeader_1.27mm:PinHeader_2x10_P1.27mm_Vertical_SMD -> Connector_PinSocket_1.27mm:PinSocket_2x10_P1.27mm_Vertical_SMD
Changed lines of the file:
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@@
 			)
 		)
-		(property "Footprint" "Connector_PinHeader_1.27mm:PinHeader_2x10_P1.27mm_Vertical_SMD"
+		(property "Footprint" "Connector_PinSocket_1.27mm:PinSocket_2x10_P1.27mm_Vertical_SMD"
 			(at 88.9 92.71 0)
 			(effects
